File: mesinCuciTangan.brd (EAGLE design)
At the start: 100 x 80 mm, 9 parts, among them X1 PIR, X2 POWER, X3 IR1, X4 IR2

Commit message: Skema Beta V0.1
Parts:
- added JP1: 12VOUTLET, pinhead:1X05
- added JP2: GNDOUTLET, pinhead:1X05
- added JP3: 5VOUTLET, pinhead:1X05
- added R1: 1K, rcl:0207/10
- added SPK_L, SPK_R: (no value), con-wago-500:W237-102
- LM2596: value CP8-ADJ -> LM2596
- renumbered U$1 to LM2596
Connections:
- removed net 5V: ARDUINO_NANO1.12
- new net +12V: JP1.1, JP1.2, JP1.3, JP1.4, JP1.5, LM2596.IN+, X2.1
- new net A0: ARDUINO_NANO1.4, U$3.4
- new net A1: ARDUINO_NANO1.5, U$3.5
- new net A2: ARDUINO_NANO1.6, U$3.6
- new net D10: ARDUINO_NANO1.28, U$2.TX
- new net D11: ARDUINO_NANO1.29, R1.1
- new net D2: ARDUINO_NANO1.20, X1.2
- new net D3: ARDUINO_NANO1.21, X3.2
- new net D4: ARDUINO_NANO1.22, X4.2
- new net N$1: MOD1.7, SPK_R.1
- new net N$2: MOD1.1, U$2.DAC_L
- new net N$3: MOD1.3, U$2.DAC_R
- new net N$4: MOD1.6, SPK_R.2
- new net N$5: MOD1.8, SPK_L.2
- new net N$6: MOD1.9, SPK_L.1
- new net N$7: R1.2, U$2.RX
- net +5V: now also ARDUINO_NANO1.12, JP3.1, JP3.2, JP3.3, JP3.4, JP3.5, LM2596.OUT+, U$2.VCC, U$3.2, X1.1, X3.1, X4.1
- net GND: now also JP2.1, JP2.2, JP2.3, JP2.4, JP2.5, LM2596.IN-, LM2596.OUT-, U$2.GND_1, U$3.3, X1.3, X2.2, X3.3, X4.3

Commit message: simple Route Without jumper
Parts:
- moved R1 268.1 mm to (102.4, 72.2), turned to 90 degrees
- moved SPK_R 250.3 mm to (77.5, 94.8)
- moved X4 245.2 mm to (142.2, 95.0), turned to 180 degrees
- moved JP2 241.5 mm to (110.4, 49.8), turned to 90 degrees
- moved JP3 237.8 mm to (104.8, 49.8), turned to 90 degrees
- moved X3 234.6 mm to (142.2, 88.5), turned to 180 degrees
- moved SPK_L 230.8 mm to (67.1, 94.8)
- moved JP1 228.9 mm to (99.1, 49.8), turned to 90 degrees
- moved U$2 215.4 mm to (100.7, 88.0), turned to 180 degrees
- moved MOD1 208.7 mm to (69.1, 66.5)
- moved ARDUINO_NANO1 170.7 mm to (135.0, 67.3)
- moved X1 162.8 mm to (142.2, 82.0), turned to 180 degrees
- moved X2 147.6 mm to (52.7, 94.9)
- moved LM2596 120.8 mm to (83.2, 28.8), turned to 270 degrees
- moved U$3 96.0 mm to (96.0, 0.00)
Connections:
- net D2: now also X1.3; no longer X1.2
- net D3: now also X3.3; no longer X3.2
- net D4: now also X4.3; no longer X4.2
- net GND: now also X1.2, X3.2, X4.2; no longer X1.3, X3.3, X4.3
Routing:
- net GND: track 0.00 -> 460.0 mm
- net +5V: track 0.00 -> 251.3 mm
- net +12V: track 0.00 -> 113.3 mm
- net N$2: track 0.00 -> 55.9 mm
- net N$3: track 0.00 -> 47.7 mm
- net D4: track 0.00 -> 22.0 mm
- net D11: track 0.00 -> 21.1 mm
- net D10: track 0.00 -> 16.2 mm
- net D3: track 0.00 -> 14.5 mm
- net A2: track 0.00 -> 14.1 mm
- net A1: track 0.00 -> 14.1 mm
- net A0: track 0.00 -> 14.1 mm
- net N$1: track 0.00 -> 13.4 mm
- net N$6: track 0.00 -> 12.5 mm
- net N$4: track 0.00 -> 11.2 mm
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Other:
- board size 100 x 80 mm -> 160 x 100 mm
- board text added: "Power Supply Place"
