File: mesinCuciTangan.brd (EAGLE design)
At the start: 160 x 100 mm, 15 parts, among them X1 PIR, X2 POWER, X3 IR1, X4 IR2

Commit message: pcb coba ceta #1
Parts:
- renumbered MOD1 to PAM8403
Routing:
- net N$8: track 0.00 -> 520.0 mm
- net GND: track 460.0 -> 457.1 mm
Other:
- board text added: "12v"
- board text added: "Buck"
- board text added: "IN- IN+"
- board text added: "OUT - OUT+"
- board text added: "Relay"
- board text added: "Tempat Power Supply"
- board text removed: "Power Supply Place"

Commit message: commit with code
Parts:
- removed SPK_L: (no value), con-wago-500:W237-102
- X3, X4: device con-molex:22-23-2031 -> con-molex:22-23-2041
- moved PAM8403 28.4 mm to (96.5, 59.1), turned to 90 degrees
- moved X2 20.3 mm to (68.1, 81.7), turned to 90 degrees
- moved X4 18.5 mm to (125.0, 88.2), turned to 270 degrees
- moved R1 16.8 mm to (113.3, 85.0)
- moved X3 8.76 mm to (133.5, 88.2), turned to 270 degrees
- moved U$2 6.66 mm to (94.0, 88.3), turned to 90 degrees
- moved X1 5.21 mm to (142.0, 87.2), turned to 270 degrees
- moved SPK_R 4.86 mm to (73.2, 92.5), turned to 90 degrees
- moved LM2596 2.24 mm to (84.2, 30.8)
- moved JP1 1.00 mm to (99.1, 48.8)
- moved JP2 1.00 mm to (110.4, 48.8)
- moved JP3 1.00 mm to (104.8, 48.8)
Connections:
- removed net N$5: PAM8403.8, SPK_L.2
- removed net N$6: PAM8403.9, SPK_L.1
- new net D5: ARDUINO_NANO1.23, X4.3
- new net D6: ARDUINO_NANO1.24, X4.4
- net D4: now also X3.4; no longer X4.3
Routing:
- net +5V: track 251.3 -> 338.9 mm
- net N$8: track 520.0 -> 440.0 mm
- net GND: track 457.1 -> 396.7 mm
- net +12V: track 113.3 -> 77.0 mm
- net D10: track 16.2 -> 49.7 mm
- net N$7: track 10.5 -> 40.0 mm
- net D5: track 0.00 -> 16.9 mm
- net N$4: track 11.2 -> 25.3 mm
- net D11: track 21.1 -> 7.65 mm
- net N$1: track 13.4 -> 26.5 mm
- net N$6: track 12.5 -> 0.00 mm
- net D4: track 22.0 -> 10.1 mm
- net D6: track 0.00 -> 11.5 mm
- net N$3: track 47.7 -> 59.0 mm
- net N$5: track 9.13 -> 0.00 mm
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- added copper zone on layer 16, net GND
Other:
- board size 160 x 100 mm -> 120 x 100 mm
- board text removed: "Tempat Power Supply"
